File: C10/Test/c10P07d3/c10P07d3.kicad_sch (KiCad schematic)
At the start: 3 parts

Commit message: additional and moved files Chapter 10
Parts:
- removed R1: 4, symbol Device:R
- removed R2: 12, symbol Device:R
- removed V1: 20, symbol Simulation_SPICE:VDC
- added Rl3: 12, symbol Device:R
- added Rth11: 3, symbol Device:R
- added Vth1: 15, symbol Simulation_SPICE:VDC
Connections:
- net A: now also Rl3.1, Rth11.2
- net GND: now also Rl3.2, Vth1.2
- new net: Rth11.1, Vth1.1
