File: C10/Test/c10P08a/c10P08a.kicad_sch (KiCad schematic)
At the start: 3 parts

Commit message: additional and moved files Chapter 10
Parts:
- removed V1: 20, symbol Simulation_SPICE:VDC
- added R3: 680, symbol Device:R
- added Rl4: 100, symbol Device:R
- added Vt1: 120, symbol Simulation_SPICE:VDC
- R1: value 4 -> 12
- R2: value 12 -> 1.8k
Connections:
- net A: now also R3.2, Rl4.1; no longer R1.2, R2.1
- net GND: now also Rl4.2, Vt1.2
- net at R1.1: now also Vt1.1
- new net: R1.2, R2.1, R3.1
