File: C10/Test/c10P08b/c10P08b.kicad_sch (KiCad schematic)
At the start: 3 parts

Commit message: additional and moved files Chapter 10
Parts:
- removed Rl3, Rth11: 3, symbol Device:R
- removed Vth1: 15, symbol Simulation_SPICE:VDC
- added R1: 12, symbol Device:R
- added R2: 1.8k, symbol Device:R
- added R3: 680, symbol Device:R
- added Vt1: 120, symbol Simulation_SPICE:VDC
Connections:
- net A: now also R3.2
- net GND: now also R2.2, Vt1.2
- new net: R1.2, R2.1, R3.1
- new net: R1.1, Vt1.1
