File: C10/Test/c10P08c/c10P08c.kicad_sch (KiCad schematic)
At the start: 3 parts

Commit message: additional and moved files Chapter 10
Parts:
- removed Rl3: 12, symbol Device:R
- Rth11: value 3 -> 691.92
- Vth1: value 15 -> 119.2
