File: C10/Test/c10P08d/c10P08d.kicad_sch (KiCad schematic)
At the start: 3 parts

Commit message: additional and moved files Chapter 10
Parts:
- removed Rl3: 6, symbol Device:R
- added Rl4: 100, symbol Device:R
- Rth11: value 3 -> 691.92
- Vth1: value 15 -> 119.2
Connections:
- net A: now also Rl4.1
- net GND: now also Rl4.2
Changed lines of the file:
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@@
 	(paper "A4")
+	(junction
+		(at 135.89 93.98)
+		(diameter 0)
+		(color 0 0 0 0)
+	)
+	(junction
+		(at 173.99 93.98)
+		(diameter 0)
+		(color 0 0 0 0)
+	)
 	(junction
 		(at 173.99 71.12)
@@
 		(color 0 0 0 0)
 	)
-	(junction
-		(at 173.99 93.98)
-		(diameter 0)
-		(color 0 0 0 0)
-	)
-	(junction
-		(at 135.89 93.98)
-		(diameter 0)
-		(color 0 0 0 0)
+	(wire
+		(pts
+			(xy 173.99 80.01) (xy 173.99 71.12)
+		)
+		(stroke
+			(width 0)
+			(type default)
+		)
+	)
+	(wire
+		(pts
+			(xy 135.89 93.98) (xy 173.99 93.98)
+		)
+		(stroke
+			(width 0)
+			(type default)
+		)
+	)
+	(wire
+		(pts
+			(xy 135.89 93.98) (xy 135.89 100.33)
+		)
+		(stroke
+			(width 0)
+			(type default)
+		)
+	)
+	(wire
+		(pts
+			(xy 135.89 93.98) (xy 135.89 90.17)
+		)
+		(stroke
+			(width 0)
+			(type default)
+		)
+	)
+	(wire
+		(pts
+			(xy 173.99 87.63) (xy 173.99 93.98)
+		)
+		(stroke
+			(width 0)
+			(type default)
+		)
+	)
+	(wire
+		(pts
+			(xy 173.99 71.12) (xy 175.26 71.12)
+		)
+		(stroke
+			(width 0)
+			(type default)
+		)
+	)
+	(wire
+		(pts
+			(xy 135.89 71.12) (xy 144.78 71.12)
+		)
+		(stroke
+			(width 0)
+			(type default)
+		)
+	)
+	(wire
+		(pts
+			(xy 173.99 93.98) (xy 175.26 93.98)
+		)
+		(stroke
+			(width 0)
+			(type default)
+		)
 	)
 	(wire
@@
 	(wire
 		(pts
-			(xy 135.89 93.98) (xy 135.89 100.33)
-		)
-		(stroke
-			(width 0)
-			(type default)
-		)
-	)
-	(wire
-		(pts
-			(xy 173.99 71.12) (xy 175.26 71.12)
-		)
-		(stroke
-			(width 0)
-			(type default)
-		)
-	)
-	(wire
-		(pts
-			(xy 173.99 93.98) (xy 175.26 93.98)
-		)
-		(stroke
-			(width 0)
-			(type default)
-		)
-	)
-	(wire
-		(pts
 			(xy 135.89 80.01) (xy 135.89 71.12)
 		)
@@
 		)
 	)
-	(wire
-		(pts
-			(xy 173.99 80.01) (xy 173.99 71.12)
-		)
-		(stroke
-			(width 0)
-			(type default)
-		)
-	)
-	(wire
-		(pts
-			(xy 173.99 87.63) (xy 173.99 93.98)
-		)
-		(stroke
-			(width 0)
-			(type default)
-		)
-	)
-	(wire
-		(pts
-			(xy 135.89 93.98) (xy 173.99 93.98)
-		)
-		(stroke
-			(width 0)
-			(type default)
-		)
-	)
-	(wire
-		(pts
-			(xy 135.89 71.12) (xy 144.78 71.12)
-		)
-		(stroke
-			(width 0)
-			(type default)
-		)
-	)
-	(wire
-		(pts
-			(xy 135.89 93.98) (xy 135.89 90.17)
-		)
-		(stroke
-			(width 0)
-			(type default)
-		)
-	)
-	(label "B"
-		(at 175.26 93.98 0)
+	(label "A"
+		(at 175.26 71.12 0)
 		(effects
 			(font
@@
 		)
 	)
-	(label "A"
-		(at 175.26 71.12 0)
+	(label "B"
+		(at 175.26 93.98 0)
 		(effects
 			(font
@@
 			)
 		)
-		(property "Value" "15"
+		(property "Value" "119.2"
 			(at 139.7 86.2301 0)
 			(show_name no)
@@
 		)
 		(instances
-			(project "c10P07c2"
-				(path "/af3f7876-9b08-45d7-9571-4201a99e8bb2"
+			(project "c10P08d"
+				(path "/639649ce-77ca-4715-8c24-9f08f5b1e729"
 					(reference "Vth1")
 					(unit 1)
@@
 		)
 		(instances
-			(project "c10P07c2"
-				(path "/af3f7876-9b08-45d7-9571-4201a99e8bb2"
+			(project "c10P08d"
+				(path "/639649ce-77ca-4715-8c24-9f08f5b1e729"
 					(reference "#PWR01")
 					(unit 1)
@@
 		(dnp no)
 		(fields_autoplaced yes)
-		(property "Reference" "Rl3"
+		(property "Reference" "Rl4"
 			(at 176.53 82.5499 0)
 			(show_name no)
@@
 			)
 		)
-		(property "Value" "6"
+		(property "Value" "100"
 			(at 176.53 85.0899 0)
 			(show_name no)
@@
 		)
 		(instances
-			(project "c10P07c2"
-				(path "/af3f7876-9b08-45d7-9571-4201a99e8bb2"
-					(reference "Rl3")
+			(project "c10P08d"
+				(path "/639649ce-77ca-4715-8c24-9f08f5b1e729"
+					(reference "Rl4")
 					(unit 1)
 				)
@@
 			)
 		)
-		(property "Value" "3"
+		(property "Value" "691.92"
 			(at 148.59 67.31 90)
 			(show_name no)
@@
 		)
 		(instances
-			(project "c10P07c2"
-				(path "/af3f7876-9b08-45d7-9571-4201a99e8bb2"
+			(project "c10P08d"
+				(path "/639649ce-77ca-4715-8c24-9f08f5b1e729"
 					(reference "Rth11")
 					(unit 1)
