File: C10/Test/S5/f35/c10P24/c10P24.kicad_sch (KiCad schematic)
At the start: 5 parts

Commit message: additiona upload Chapter 10
Parts:
- removed R1: 12, symbol Device:R
- removed R2: 3, symbol Device:R
- removed R3: 6, symbol Device:R
- removed V1: 84, symbol Simulation_SPICE:VDC
- removed V2: 21, symbol Simulation_SPICE:VDC
- added In1: 5, symbol Simulation_SPICE:IDC
- added Rl3, Rn1: 6, symbol Device:R
Connections:
- net A: now also In1.2, Rl3.1, Rn1.1
- net GND: now also In1.1, Rl3.2, Rn1.2
