File: C10/Test/S7/f38/c10P32/c10P32.kicad_sch (KiCad schematic)
At the start: 5 parts

Commit message: additiona upload Chapter 10
Parts:
- removed V1: 84, symbol Simulation_SPICE:VDC
- removed V2: 21, symbol Simulation_SPICE:VDC
- added Vt1: 20, symbol Simulation_SPICE:VDC
- added Vt2: 40, symbol Simulation_SPICE:VDC
- R1: value 12 -> 10
- R2: value 3 -> 10
- R3: value 6 -> 15
Connections:
- net GND: now also Vt1.2, Vt2.2
- net at R1.1: now also Vt1.1
- net at R2.2: now also Vt2.1
