File: C10/Test/S7/f38/c10P32a/c10P32a.kicad_sch (KiCad schematic)
At the start: 5 parts

Commit message: additiona upload Chapter 10
Parts:
- removed V1: 84, symbol Simulation_SPICE:VDC
- removed V2: 21, symbol Simulation_SPICE:VDC
- added I1: 2, symbol Simulation_SPICE:IDC
- added I2: 4, symbol Simulation_SPICE:IDC
- R1: value 12 -> 10
- R2: value 3 -> 10
- R3: value 6 -> 15
Connections:
- net A: now also R2.2, I1.2, I2.2; no longer R2.1
- net GND: now also R1.1, R2.1, I1.1, I2.1
