File: C10/Test/S2/f28/c10P09a1/c10P09a1.kicad_sch (KiCad schematic)
At the start: 5 parts

Commit message: corrected from misprinting Fig 10-28
Parts:
- R1: value 12 -> 1.2k
Changed lines of the file:
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@@
 			)
 		)
-		(property "Value" "12"
+		(property "Value" "1.2k"
 			(at 148.59 66.04 90)
 			(show_name no)
