File: C10/Test/S9/c10P41a/c10P41a.kicad_sch (KiCad schematic)
At the start: 6 parts

Commit message: corrected due to misprinting Fig 10-45
Parts:
- R1, R4: value 10k -> 10
Changed lines of the file:
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@@
 			)
 		)
-		(property "Value" "10k"
+		(property "Value" "10"
 			(at 165.1 92.7099 0)
 			(show_name no)
@@
 			)
 		)
-		(property "Value" "10k"
+		(property "Value" "10"
 			(at 203.2 80.0099 0)
 			(show_name no)
