File: C34/Lecture/c34F19/c34F19.kicad_sch (KiCad schematic)
At the start: 14 parts

Commit message: Additional Test in Chapter 34
Parts:
- Rdt8: value 7.55k -> 5k
Changed lines of the file:
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@@
 			)
 		)
-		(property "Value" "7.55k"
+		(property "Value" "5k"
 			(at 69.85 100.3299 0)
 			(show_name no)
