File: C34/Lecture/c34F27/c34F27.kicad_sch (KiCad schematic)
At the start: 6 parts, among them U1 ${SIM.PARAMS}

Commit message: Additional Test in Chapter 34
Connections:
- net Vout1: now reaches D1.2 (A), U1.5
- net Vout renamed Vout2
Changed lines of the file:
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@@
+	)
+	(junction
+		(at 186.69 82.55)
+		(diameter 0)
+		(color 0 0 0 0)
 	)
 	(junction
@@
 	(wire
 		(pts
-			(xy 182.88 82.55) (xy 190.5 82.55)
+			(xy 182.88 82.55) (xy 186.69 82.55)
 		)
 		(stroke
@@
 	(wire
 		(pts
+			(xy 186.69 82.55) (xy 190.5 82.55)
+		)
+		(stroke
+			(width 0)
+			(type default)
+		)
+	)
+	(wire
+		(pts
 			(xy 143.51 80.01) (xy 143.51 83.82)
 		)
@@
 		(pts
 			(xy 138.43 80.01) (xy 143.51 80.01)
+		)
+		(stroke
+			(width 0)
+			(type default)
+		)
+	)
+	(wire
+		(pts
+			(xy 186.69 72.39) (xy 186.69 82.55)
 		)
 		(stroke
@@
 		)
 	)
-	(label "Vout"
+	(label "Vout2"
 		(at 215.9 82.55 0)
 		(effects
 			(font
+				(size 1.27 1.27)
+			)
+			(justify left bottom)
+		)
+	)
+	(label "Vout1"
+		(at 186.69 72.39 0)
+		(effects
+			(font
