File: C34/Lecture/c34F28/c34F28.kicad_sch (KiCad schematic)
At the start: 7 parts, among them U1 ${SIM.PARAMS}

Commit message: Additional Test in Chapter 34
Connections:
- net Vout1: now reaches D1.2 (A), U1.5
- net Vout renamed Vout2
Changed lines of the file:
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@@
+	)
+	(junction
+		(at 186.69 83.82)
+		(diameter 0)
+		(color 0 0 0 0)
 	)
 	(junction
@@
 	(wire
 		(pts
+			(xy 186.69 73.66) (xy 186.69 83.82)
+		)
+		(stroke
+			(width 0)
+			(type default)
+		)
+	)
+	(wire
+		(pts
 			(xy 172.72 111.76) (xy 110.49 111.76)
 		)
@@
 	(wire
 		(pts
+			(xy 186.69 83.82) (xy 190.5 83.82)
+		)
+		(stroke
+			(width 0)
+			(type default)
+		)
+	)
+	(wire
+		(pts
 			(xy 110.49 81.28) (xy 110.49 86.36)
 		)
@@
 	(wire
 		(pts
-			(xy 182.88 83.82) (xy 190.5 83.82)
+			(xy 182.88 83.82) (xy 186.69 83.82)
 		)
 		(stroke
@@
 		)
 	)
-	(label "Vout"
+	(label "Vout2"
 		(at 223.52 83.82 0)
 		(effects
@@
 		)
 	)
+	(label "Vout1"
+		(at 186.69 73.66 0)
+		(effects
+			(font
+				(size 1.27 1.27)
+			)
+			(justify left bottom)
+		)
+	)
